File: kicad/main/main2.kicad_pcb (KiCad board)
At the start: 2 copper layers, 30.7 x 51.3 mm, 68 parts, among them J2 U.FL-R-SMT_01_, P1 USB_C_Plug_USB2.0, SW1 SW_Push, U1 AMS1117-3.3, U2 ESP32-S3-WROOM-1, U3 AXP2101, U4 ZOE-M8Q, U5 BNO080, Y1 32.768Khz Crystal, Y2 32.768Khz Crystal

Commit message: added mainbase
Parts:
- added G***: LOGO, LOGO, F.Cu at (104.9, 88.3)
- C21, C4: moved to F.Cu
- R8: moved to B.Cu
- moved C21 3.14 mm to (112.6, 87.8), turned to 90 degrees
- moved R8 0.54 mm to (110.9, 83.8), turned to 180 degrees
- turned C4 to 0 degrees
Other:
- board text removed: "TRAX"

Commit message: changed vis
Parts:
- moved G*** 0.40 mm to (105.0, 87.9)
